File: trunk/PCB/main_board/main_board.kicad_pcb (KiCad board)
At the start: 2 copper layers, 190 x 142 mm, 52 parts, among them J1 POWER, J2 LCD_SC2004, J3 SPI7SEG, J4 Conn_01x05, J5 Conn_01x05, J6 Conn_01x05, J7 Conn_01x05, SW1 SW_UP, SW2 SW_DOWN, SW3 SW_OK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

Commit message: RTCのバックアップ電源ラインに逆流防止ダイオードが抜けていたのを追加 タクトスイッチのフットプリントが間違っていたのを修正
git-svn-id: https://shiro-home.ddns.net/svn/project/date-counter@12 7e553844-23e9-431f-8cc1-739bbe1f3d25
Parts:
- added D2: 1N4148, Diode_THT:D_DO-15_P10.16mm_Horizontal, F.Cu at (239.4, 143.7)
- turned SW5 to 0 degrees
Connections:
- D1 pad 1: +5V -> Net-(D1-Pad1)
- U2 pad 8: +5V -> Net-(D1-Pad1)
Routing:
- net Net-(D1-Pad1): track 0.00 -> 27.9 mm
- net +5V: track 244.3 -> 236.1 mm
- net /SW_OK2: track 19.8 -> 14.2 mm
- net /SW_CANCEL2: track 39.3 -> 34.8 mm
- net /SW_UP2: track 32.4 -> 36.3 mm
- net /SW_DOWN2: track 11.4 -> 15.2 mm
- net /RESET2: track 114.3 -> 116.3 mm
- net GND: track 50.3 -> 52.2 mm
Other:
- outline, holes or cut-outs redrawn
