File: trunk/PCB/main_board/main_board.sch (KiCad schematic (older format))
At the start: 24 parts, among them J1 POWER, J2 LCD_SC2004, J3 SPI7SEG, J4 Conn_01x05, J5 Conn_01x05, J6 Conn_01x05, J7 Conn_01x05, SW1 SW_UP, SW2 SW_DOWN, SW3 SW_OK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

Commit message: RTCのバックアップ電源ラインに逆流防止ダイオードが抜けていたのを追加 タクトスイッチのフットプリントが間違っていたのを修正
git-svn-id: https://shiro-home.ddns.net/svn/project/date-counter@12 7e553844-23e9-431f-8cc1-739bbe1f3d25
Parts:
- added D2: 1N4148, Diode_THT:D_DO-15_P10.16mm_Horizontal, symbol Device:D
- U1: symbol MyLib2:DaVinci_32U -> main_board-rescue:DaVinci_32U-MyLib2
- U2: symbol MyLib2:AE-RX8025 -> main_board-rescue:AE-RX8025-MyLib2
Connections:
- net +5V: now also D2.2 (A); no longer D1.1 (K), U2.8 (VDD)
- new net: D1.1 (K), D2.1 (K), U2.8 (VDD)
Changed lines of the file:
@@
 $EndDescr
 $Comp
-L MyLib2:DaVinci_32U U1
+L main_board-rescue:DaVinci_32U-MyLib2 U1
 U 1 1 60D9351C
 P 5400 2500
@@
 $EndComp
 $Comp
-L MyLib2:AE-RX8025 U2
+L main_board-rescue:AE-RX8025-MyLib2 U2
 U 1 1 60D9FE06
 P 9750 3500
@@
 L power:+5V #PWR014
 U 1 1 60DAF7B7
-P 9150 3200
-F 0 "#PWR014" H 9150 3050 50  0001 C CNN
-F 1 "+5V" H 9165 3373 50  0000 C CNN
-F 2 "" H 9150 3200 50  0001 C CNN
-F 3 "" H 9150 3200 50  0001 C CNN
-	1    9150 3200
+P 8750 3000
+F 0 "#PWR014" H 8750 2850 50  0001 C CNN
+F 1 "+5V" H 8765 3173 50  0000 C CNN
+F 2 "" H 8750 3000 50  0001 C CNN
+F 3 "" H 8750 3000 50  0001 C CNN
+	1    8750 3000
 	1    0    0    -1
 $EndComp
@@
 Text Label 2550 6000 2    50   ~ 0
 SW_UP2
+$Comp
+L Device:D D2
+U 1 1 61EE892D
+P 9000 3200
+F 0 "D2" H 9000 3417 50  0000 C CNN
+F 1 "1N4148" H 9000 3326 50  0000 C CNN
+F 2 "Diode_THT:D_DO-15_P10.16mm_Horizontal" H 9000 3200 50  0001 C CNN
+F 3 "~" H 9000 3200 50  0001 C CNN
+	1    9000 3200
+	-1   0    0    -1
+$EndComp
+Wire Wire Line
+	8750 3000 8750 3200
+Wire Wire Line
+	8750 3200 8850 3200
 $EndSCHEMATC
